File: Tanimoji-PCB/Tanimoji-PCB.kicad_pcb (KiCad board)
At the start: 2 copper layers, 67 parts, among them J1 Battery Connector, J2 Screw_Terminal_01x04, J3 Screw_Terminal_01x07, J4 Screw_Terminal_01x04, J5 Screw_Terminal_01x03, J6 Screw_Terminal_01x02, J7 Conn_01x01_Pin, J8 Conn_01x01_Pin, Q1 BSS138, Q2 BSS138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

Commit message: -
Parts:
- removed J4: Screw_Terminal_01x04, Connector_JST:JST_XH_B4B-XH-AM_1x04_P2.50mm_Vertical
- added REF**: TestPoint_Pad_1.0x1.0mm, TestPoint:TestPoint_Pad_1.0x1.0mm, B.Cu at (152.8, 90.1)
- added REF**: TestPoint_Pad_1.0x1.0mm, TestPoint:TestPoint_Pad_1.0x1.0mm, B.Cu at (156.1, 90.1)
- added REF**: TestPoint_Pad_1.0x1.0mm, TestPoint:TestPoint_Pad_1.0x1.0mm, B.Cu at (157.8, 90.1)
- added REF**: TestPoint_Pad_1.0x1.0mm, TestPoint:TestPoint_Pad_1.0x1.0mm, B.Cu at (154.4, 90.1)
- added mouse-bite-2.54mm-slot: VAL**, mousbites:mouse-bite-2.54mm-slot, F.Cu at (155.1, 69.0)
- JP1, JP10, JP2, JP3, JP4, JP5, JP6, JP7, JP8, JP9: moved to B.Cu
- moved C5 74.5 mm to (173.2, 55.1), turned to 180 degrees
- moved J8 70.9 mm to (116.9, 101.6)
- moved C4 63.3 mm to (162.2, 55.9), turned to -90 degrees
- moved JP7 61.5 mm to (159.6, 108.6), turned to -90 degrees
- moved C1 60.1 mm to (166.2, 60.1), turned to -90 degrees
- moved JP3 58.3 mm to (173.5, 63.1), turned to 180 degrees
- moved JP8 57.2 mm to (162.2, 108.6), turned to -90 degrees
- moved R10 57.0 mm to (173.2, 57.1), turned to 180 degrees
- moved J2 55.1 mm to (136.6, 46.9)
- moved R9 54.1 mm to (173.2, 59.2)
- moved C3 54.0 mm to (149.3, 51.8), turned to -90 degrees
- moved R3 52.6 mm to (171.9, 64.4)
- moved R8 51.7 mm to (173.2, 60.9)
- moved R5 51.4 mm to (166.2, 62.8), turned to 180 degrees
- moved R4 50.8 mm to (168.4, 64.4), turned to 180 degrees
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Routing:
- net +3.3V: track 0.00 -> 189.7 mm, vias 0 -> 8
- net +5V: track 0.00 -> 105.5 mm, vias 0 -> 5
- net ESP_TX2: track 0.00 -> 82.2 mm, vias 0 -> 1
- net ESP_RX2: track 0.00 -> 82.1 mm, vias 0 -> 1
- net TOUCH_2: track 0.00 -> 78.4 mm
- net ESP_EN: track 0.00 -> 76.9 mm, vias 0 -> 2
- net ESP_RX: track 0.00 -> 74.9 mm, vias 0 -> 2
- net ESP_CLK: track 0.00 -> 70.3 mm, vias 0 -> 1
- net ESP_TX: track 0.00 -> 69.8 mm, vias 0 -> 3
- net ESP_MOSI: track 0.00 -> 65.9 mm, vias 0 -> 1
- net GND: track 0.00 -> 59.2 mm, vias 0 -> 63
- net TFT_CS: track 0.00 -> 57.1 mm, vias 0 -> 3
- net Net-(JP4-B): track 0.00 -> 54.9 mm, vias 0 -> 2
- net TFT_RST: track 0.00 -> 53.5 mm, vias 0 -> 1
- net SCL: track 0.00 -> 43.2 mm
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- added copper zone on B.Cu, net GND
- added copper zone on F.Cu, net GND
- added copper zone on In1.Cu, net GND
- added copper zone on In2.Cu, net GND
- added copper zone on B.Cu, net GND2
- added copper zone on F.Cu, net GND2
- added copper zone on In1.Cu, net GND2
- added copper zone on In2.Cu, net GND2
Other:
- board outline added: 90 x 80.8 mm
- copper layers 2 -> 4
- board text added: "*"
- board text added: "+"
- board text added: "-"
- board text added: "1"
- board text added: "2"
- board text added: "3.3V"
- board text added: "3V3"
- board text added: "ADC"
- board text added: "BAT"
- board text added: "BOOT0"
- board text added: "CLK"
- board text added: "CS"
- board text added: "DC"
- board text added: "GND"
- board text added: "LCD"
- board text added: "MOSI"
- board text added: "RESET"
- board text added: "RST"
- board text added: "RX"
- board text added: "SCL"
- board text added: "SDA"
- board text added: "SPKR"
- board text added: "TX"
- board text added: "VCC"
